File: Metronome/Metronome.kicad_pcb (KiCad board)
At the start: 2 copper layers, 68.6 x 36.2 mm, 53 parts, among them P1 CONN_01X02, P3 CONN_01X05, SW1 SW_PUSH, SW2 SW_PUSH, SW3 SW_PUSH, SW4 SW_PUSH, SW5 SW_PUSH, SW7 SWITCH_INV, T1 BSS138, T2 BSS83P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

Commit message: Deleting unnecessary traces on PCB
Parts:
- removed R10, R7: 100, Resistors_SMD:R_0603_HandSoldering
- removed R19: TODO, Resistors_SMD:R_0805_HandSoldering
- removed R8, R9: 470K, Resistors_SMD:R_0603_HandSoldering
- removed REF** (x4): 1pin, Connect:1pin
- removed REF***: OSHW-Logo2_7.3x6mm_Copper, Symbols:OSHW-Logo2_7.3x6mm_Copper
- removed T2, T5: BSS83P, TO_SOT_Packages_SMD:SOT-23_Handsoldering
- removed T3, T6: BSS138, TO_SOT_Packages_SMD:SOT-23_Handsoldering
Connections:
- P1 pad 1: Net-(P1-Pad1) -> VCC
- P1 pad 2: SNDOUT2 -> Net-(P1-Pad2)
- T4 pad 3: Net-(T3-Pad2) -> Net-(P1-Pad2)
- U2 pad 8: SNDTIMER2 -> Net-(U2-Pad8)
- U2 pad 9: SNDTIMER1 -> Net-(U2-Pad9)
Routing:
- net SNDTIMER1: track 32.2 -> 0.00 mm
- net SNDOUT2: track 26.8 -> 0.00 mm, vias 2 -> 0
- net SNDTIMER2: track 24.4 -> 0.00 mm
- net Net-(T3-Pad2): track 20.0 -> 0.00 mm
- net SNDOUT1: track 14.8 -> 0.00 mm, vias 1 -> 0
- net VCC: track 222.4 -> 209.3 mm, vias 8 -> 6
- net Net-(R10-Pad2): track 8.99 -> 0.00 mm
- net Net-(R7-Pad1): track 8.99 -> 0.00 mm
- net Net-(P1-Pad1): track 3.48 -> 0.00 mm

Commit message: Fixes on PCB
New PCB version is not yet ready.
Parts:
- U2: footprint SMD_Packages:SSOP-20 -> Housings_SSOP:SSOP-20_5.3x7.2mm_Pitch0.65mm
- moved X1 19.4 mm to (64.5, 208.5)
- moved U2 15.1 mm to (49.8, 204.3), turned to 180 degrees
Routing:
- net GND: track 512.6 -> 468.9 mm, vias 49 -> 43
- net PWMOUT: track 51.3 -> 42.4 mm, vias 2 -> 0
- net DISPLAYENABLE: track 19.2 -> 12.6 mm
- net CLKOUT: track 3.23 -> 0.00 mm
- net ICSPDAT: track 47.4 -> 44.6 mm
- net VCC: track 209.3 -> 206.5 mm
- net BUT1MCU: track 16.5 -> 18.4 mm
- net BUT2MCU: track 17.6 -> 19.1 mm
- net ICPSCLK: track 48.6 -> 47.3 mm
- net BUT4MCU: track 20.7 -> 21.8 mm
- net BUT5MCU: track 16.7 -> 17.8 mm
- net BUT3MCU: track 19.4 -> 20.5 mm
- net METRONOME: track 11.0 -> 12.0 mm
- net RESET: track 22.9 -> 22.1 mm
